File: KiCad like a pro project 3 - uC Datalogger/KiCad like a pro project 3 - uC Datalogger.kicad_sch (KiCad schematic)
At the start: 25 parts, among them U1 24LC1025, U2 24LC1025, U3 DS1337S+, U4 ATMEGA328P_VQFNVQFN, Y1 32.768 KHz, Y2 16 MHz

Commit message: enh layout and text schematic
Other:
- title: &(project_name) -> MCU Datalogger
Changed lines of the file:
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@@
   (paper "A4")
   (title_block
-    (title "&(project_name)")
-    (date "2022-07-29")
-    (rev "1")
+    (title "MCU Datalogger")
+    (date "2022-07-31")
+    (rev "V1.0")
+    (comment 1 "Casper Tak")
   )
   (junction (at 207.264 54.864) (diameter 0) (color 0 0 0 0)
